File: jtagger.sch (KiCad schematic (older format))
At the start: 104 parts, among them J1 µUSB, J2 ARM_JTAG, J3 PADS, Q1 IRLML6402, Q2 IRLML6402, Q3 MMBT3906, Q4 2N7002, U1 MCP1700T-3302E/TT, U10 TPS61045DRB, U11 SI8642, U2 SI8645, U3 FT2232HQ, U4 EPM240T100C5N, U5 MCP1700T-3302E/TT, U6 REE-0505S, U7 OSC-50MHz, U8 LTC1844ES5-3.3, U9 DG449DS, X1 12 MHz

Commit message: Version submitted to fab
Parts:
- removed C24, C25, C26, C27, C4: 10u, IPC7351-Nominal:CAPC2012X70, symbol C-0805
- removed DZ2, DZ3: 1SMA5914BT3G, IPC7351-Nominal:DIOM5226X203, symbol 1SMA59xxBT3G
- removed Q3: MMBT3906, smd-semi:SOT-23, symbol MMBT3906
- removed Q4: 2N7002, smd-semi:SOT-23, symbol 2N7002
- removed R11: 220k, IPC7351-Nominal:RESC1005X40, symbol R-0402
- removed R25: 1k, IPC7351-Nominal:RESC1005X40, symbol R-0402
- removed R32: 3k3, IPC7351-Nominal:RESC1005X40, symbol R-0402
- removed U1, U5: MCP1700T-3302E/TT, smd-semi:SOT-23, symbol MCP1700T-vv02E/TT
- removed U11: SI8642, IPC7351-Nominal:SOP63P600X160-16, symbol SI8642-QSOP
- removed U2: SI8645, IPC7351-Nominal:SOP63P600X160-16, symbol SI8640-QSOP
- removed U4: EPM240T100C5N, IPC7351-Nominal:QFP50P1600X1600X160-100, symbol EPM240-TQFP100
- removed U6: REE-0505S, manuf:RECOM-REE-0505S, symbol REE-0505S
- removed U8: LTC1844ES5-3.3, smd-semi:SOT-23-5, symbol LTC1844ES5-v.v
- added C24, C4, C41, C45: 1u, IPC7351-Nominal:CAPC1608X55, symbol C-0603
- added C25, C26, C27, C42, C43, C46, C47: 100n, IPC7351-Nominal:CAPC1005X55, symbol C-0402
- added J4: JTAG, conn-molex:CONN-MOLEX-52808-0871, symbol CONN-MOLEX-52808-0871
- added JP1: PROGB, symbol JUMPER-SOLDER
- added R25: THERM, IPC7351-Nominal:RESC2012X50, symbol THERM
- added R35: 10k, IPC7351-Nominal:RESC1005X40, symbol R-0402
- added TP1, TP3, TP4, TP5: DONE, conn-test:TEST-SMD-SMALL, symbol TESTPOINT
- added TP2: INITB, conn-test:TEST-SMD-SMALL, symbol TESTPOINT
- added U1: XC3S50-VQ100, IPC7351-Nominal:QFP50P1600X1600X100-100, symbol XC3S50-VQ100
- added U2: ADP322ACPZ-145, IPC7351-Nominal:QFN50P300X300X100-17, symbol ADP322
- added U4: S25FL204, IPC7351-Nominal:SOIC127P600X175-8, symbol SST25VF
- added U5: LTC1844ES5-3.3, smd-semi:SOT-23-5, symbol LTC1844ES5-v.v
- added U6: TXB0104RGY, manuf:TEXAS-RGY, symbol TXB0104RGY
- C7: value 100p -> 1u; BOM CAP MLCC 100pF C0G 16V 1% [0603] -> CAP MLCC 1u ≥X5R 10V 20% [0603]
- C9: value 1n -> 1u; BOM CAP MLCC 1n C0G 16V 1% [0603] -> CAP MLCC 1u ≥X5R 10V 20% [0603]
- J3: value PADS -> FLASH
- R12: value 1k -> 10k
- R24, R8: value 1M -> 0R; BOM RES SMD 1M 5% [0402] -> RES SMD 0 [0402]
- R26, R27: value 3k3 -> 0R; BOM RES SMD 3k3 5% [0402] -> RES SMD 0 [0402]
- R28, R29, R31: value 3k3 -> 1k; BOM RES SMD 3k3 5% [0402] -> RES SMD 1k 5% [0402]
- gave numbers to parts that had none: 2
Connections:
- net (+5) is gone; now on net +5: U10.2 (VIN)
- net CPLD_SEL is gone; now on net +3.3: R31.1
- net IN_CPLD_TDO is gone; now on an unnamed net: U3.40 (BDBUS2)
- net IN_CPLD_TMS is gone; now on an unnamed net: U3.41 (BDBUS3)
- net PC_TCK is gone; now on net +3.3: R30.1
- net TARG_#TRST is gone; now on an unnamed net: R14.2
- net TARG_TCLKO is gone; now on net IN_TCK: R17.2
- net TARG_TDI is gone; now on net IN_TDI: R15.2
- net TARG_TDO is gone; now on net IN_TDO: R19.2
- net TARG_TMS is gone; now on net IN_TMS: R16.2
- net +3.3: now also C23.1, C29.1, C31.1, C35.1, C36.1, C37.1, C38.1, C40.1, C9.1, J3.2, U7.1 (OE), U7.4 (VCC), C47.1, J4.1, TP3.1, U1.19 (VCCO_6), U1.26 (M2), U1.31 (VCCO_5), U1.46 (VCCO_4), U1.57 (VCCO_3), U1.6 (VCCO_7), U1.83 (VCCO_1), U1.94 (VCCO_0), U1.98 (HSWAP_EN), U2.5 (VOUT1), U4.3 (#WP), U4.7 (#HOLD), U4.8 (VDD), U6.1 (VCCA); no longer C39.1
- net +5: now also C41.1, U2.1 (EN1), U2.10 (VIN3), U2.15 (EN3), U2.16 (EN2), U2.2 (VBIAS), U2.3 (VIN1/2)
- net GND: now also C16.2, C17.2, C23.2, C28.2, C29.2, C30.2, C31.2, C32.2, C33.2, C34.2, C35.2, C36.2, C37.2, C38.2, C40.2, C7.2, C9.2, DS3.1, J2.10, J2.12, J2.14, J2.16, J2.18, J2.20, J2.4, J2.6, J2.8, J3.4, J3.6, J3.8, Q2.1, R23.2, R28.2, R33.2, U10.6 (GND), U10.7 (PGND), U10.9 (PGND(EP)), U7.2 (GND), U9.3 (GND), U9.7 (V-), C24.2, C25.2, C26.2, C27.2, C4.2, C41.2, C42.2, C43.2, C45.2, C46.2, C47.2, J4.3, J4.5, J4.7, JP1.2, R35.2, U1.10 (GND), U1.20 (GND), U1.24 (M1), U1.25 (M0), U1.29 (GND), U1.3 (GND), U1.41 (GND), U1.66 (GND), U1.73 (GND), U1.82 (GND), U1.95 (GND), U2.12 (GND), U2.17 (GND(EP)), U4.4 (VSS), U6.15 (EP), U6.7 (GND); no longer R8.1
- net IN_TCK: now also U1.67 (IO); no longer U3.16 (ADBUS0), U3.38 (BDBUS0)
- net IN_TDI: now also U1.64 (IO/VREF); no longer U3.17 (ADBUS1)
- net IN_TDO: now also U1.71 (IO); no longer U3.18 (ADBUS2)
- net IN_TMS: now also U1.65 (IO); no longer C7.1, C9.1, U3.19 (ADBUS3)
- net VCTRL: now also U1.1 (IO-VRN)
- net AD4: now reaches U3.21 (ADBUS4)
- net AD4: now also U1.87 (IO/GCLK4)
- net AD5: now reaches U3.22 (ADBUS5)
- net AD5: now also U1.86 (IO/VREF)
- net AD6: now reaches U3.23 (ADBUS6)
- net AD6: now also U1.85 (IO)
- net AD7: now reaches U3.24 (ADBUS7)
- net AD7: now also U1.81 (IO)
- net AD8: now reaches U3.26 (ACBUS0)
- net AD9: now reaches U3.27 (ACBUS1)
- net AD9: now also U1.80 (IO-VRP)
- net AD10: now reaches U3.28 (ACBUS2)
- net AD10: now also U1.79 (IO-VRN)
- net AD11: now reaches U3.29 (ACBUS3)
- net AD15: now reaches U3.34 (ACBUS7)
- net TGTSENSE: now reaches R12.1
- net TGTSENSE: now also U1.28 (IO/RDWR); no longer C7.2
- net CCLK: now reaches J3.1
- net CCLK: now also U1.52 (CCLK), U4.6 (CLK)
- net SPIMOSI: now reaches J3.3
- net SPIMOSI: now also U1.40 (IO/DOUT/BUSY), U4.5 (SI)
- net SPI#CS: now reaches J3.5
- net SPI#CS: now also U1.27 (IO/CS), U4.1 (#CS)
- net SPIMISO: now reaches J3.7
- net SPIMISO: now also U1.48 (IO/D0/DIN), U4.2 (SO)
- net FPGA_TCK: now reaches R28.1
- net FPGA_TCK: now also R8.1, J4.8, U1.77 (TCK); no longer Q2.1
- net at R26.2: no longer R27.1
- net +1.2: now reaches C28.1
- net +1.2: now also C27.1, C4.1, C42.1, C43.1, TP5.1, U1.18 (VCCINT(1.2V)), U1.45 (VCCINT(1.2V)), U1.69 (VCCINT(1.2V)), U1.93 (VCCINT(1.2V)), U2.8 (VOUT3)
- net at R8.2: now also U3.38 (BDBUS0); no longer R24.1
- removed net (+3.3): C17.1, C23.1, C31.1, C35.1, C36.1, C37.1, C38.1, C40.1, Q2.2, R26.1, U7.1 (OE), U7.4 (VCC)
- net (+VTGT) renamed +2.5
- net +2.5: now also C7.1, R29.1, C25.1, C26.1, TP4.1, U1.33 (VCCAUX(2.5V)), U1.58 (VCCAUX(2.5V)), U1.7 (VCCAUX(2.5V)), U1.84 (VCCAUX(2.5V)), U2.6 (VOUT2); no longer C29.1, Q2.3
- removed net (GND): C16.2, C17.2, C23.2, C28.2, C29.2, C30.2, C31.2, C32.2, C33.2, C34.2, C35.2, C36.2, C37.2, C38.2, C40.2, DS3.1, J2.10, J2.12, J2.14, J2.16, J2.18, J2.20, J2.4, J2.6, J2.8, R23.2, R24.2, R28.2, R29.2, R30.2, R31.2, R33.2, U10.6 (GND), U10.7 (PGND), U10.9 (PGND(EP)), U7.2 (GND), U9.3 (GND), U9.7 (V-)
- net 50MHz renamed 50MHZ
- net 50MHZ: now also U1.90 (IO/GCK7)
- net AUX1_HVP: no longer names the net of U9.1
- net AUX1_HVP: no longer R18.2
- net AUX1_LV: no longer names the net of U9.2
- net AUX1_LV: now also U6.13 (B1)
- net HVPEN renamed VPPEN
- net VPPEN: now also U1.15 (IO)
- net IN_CPLD_SEL renamed AD12
- net AD12: now also U1.96 (IO-VRN)
- net IN_CPLD_TDI: no longer names the net of U3.39 (BDBUS1)
- net IN_CPLD_TDI: now also R24.2
- net PULSE_LONG renamed AD13
- net PULSE_SHORT renamed +VTGT
- net +VTGT: now also C16.1, C39.1, C45.1, R25.2, R35.1, U5.2 (GND), U6.14 (VCCB); no longer U3.33 (ACBUS6)
- net TARG_#SRST: no longer names the net of R20.2
- net TARG_#SRST: now also U6.12 (B2)
- net TARG_DBGACK: no longer names the net of R22.2
- net TARG_DBGACK: now also U6.10 (B4)
- net TARG_DBGREQ: no longer names the net of R21.2
- net TARG_DBGREQ: now also U6.11 (B3)
- removed net VT_IN: C16.1, J2.1, R29.1
- new net: J2.1, Q2.3
- new net: TP2.1, U1.42 (IO/INIT)
- new net: JP1.1, R29.2, U1.99 (PROG)
- new net: Q2.2, R25.1
- new net AD0: U1.89 (IO/GCK6), U3.16 (ADBUS0)
- new net AD1: U1.92 (IO), U3.17 (ADBUS1)
- new net AD14: U3.33 (ACBUS6)
- new net AD2: U1.91 (IO/VREF), U3.18 (ADBUS2)
- new net AD3: U1.88 (IO/GCLK5), U3.19 (ADBUS3)
- new net BUFOE: U1.16 (IO/VREF), U6.8 (OE)
- new net DONE: TP1.1, U1.51 (DONE)
- new net FPGA_TDI: J4.2, R24.1, R31.2, U1.100 (TDI)
- new net FPGA_TDO: J4.4, R26.1, U1.76 (TDO)
- new net FPGA_TMS: J4.6, R27.1, R30.2, U1.78 (TMS)
- new net IN_#SRST: U1.22 (IO-VRN), U6.3 (A2)
- new net IN_#TRST: U1.23 (IO-VRP), U6.2 (A1)
- new net IN_DBGACK: U1.17 (IO), U6.5 (A4)
- new net IN_DBGREQ: U1.21 (IO), U6.4 (A3)
- new net IN_RTCK: R18.2, U1.68 (IO)
- new net VTGTLIM: C17.1, C24.1, U1.70 (VCCO_2)
- no-connect marks 4 -> 7
Other:
- note added: "Leave traces\nto allow cutting"
- note removed: "ISOLATION"
- note removed: "Static charge\ndissipative resistors"
- moved on the sheet: C16, C22, C23, C29, C30, C31, C32, C33, C34, C35, C36, C37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

Commit message: Schematic stuff
Parts:
- E1: Description (none) -> BEAD FERRITE 1000 OHM 100MA 1608
- J1: Description (none) -> CONN USB MICRO B RECPT SMT R/A
- R12, R35: BOM RES SMD 1k 5% [0402] -> RES SMD 10k 5% [0402]
- R25: value THERM -> 100mA; BOM (none) -> DIST DIGIKEY 507-1516-1-ND; Description (none) -> PTC RESTTBLE 0.10A 15V CHIP 0805; Manuf (none) -> Bel Fuse; PN (none) -> 0ZCE0010FF2G
- TP3: value DONE -> 3V3
- TP4: value DONE -> 2V5
- TP5: value DONE -> 1V2
- U1: value XC3S50-VQ100 -> XC3S50A-4VQG100C
- U5: BOM (none) -> DIST DIGIKEY LTC1844ES5-3.3#TRMPBFCT-ND; Description (none) -> IC REG LDO 3.3V 0.15A TSOT23-5; PN LTC1844ES5-v.v -> LTC1844ES5-3.3
Connections:
- net AD12: no longer U3.30 (ACBUS4)
- net SHIFT_#TRST: now reaches R14.2, U9.1
- net SHIFT_#SRST: now reaches R20.2, U6.12 (B2)
- net SHIFT_DBGREQ: now reaches R21.2, U6.11 (B3)
- net SHIFT_DBGACK: now reaches R22.2, U6.10 (B4)
- net PROGB: now reaches JP1.1, R29.2, U1.99 (PROG)
- net AD10 renamed AC2
- net AD11: no longer names the net of U3.29 (ACBUS3)
- net AD13: no longer names the net of U3.32 (ACBUS5)
- net AD14: no longer names the net of U3.33 (ACBUS6)
- net AD15: no longer names the net of U3.34 (ACBUS7)
- net AD8: no longer names the net of U3.26 (ACBUS0)
- net AD9 renamed AC1
- net DONE: no longer names the net of TP1.1, U1.51 (DONE)
- no-connect marks 7 -> 4
Other:
- note added: "FPGA MANAGEMENT"
- note added: "LEVEL-SHIFTED"
- note added: "PC DATA"
- note added: "SIGNALS TO PORT"
- note added: "SYSTEM CONTROL"
- note added: "Ultra-low dropout (30mV) regulator\nacts as voltage limiter"
- note added: "Vfb = 1.233V\nVo(min) = Vfb (@R13 / @R23 + 1) = 7.4V\nVo(max) = Vfb (@R13 / @R11 + @R13 / @R23 + 1) = 13V"
- note removed: "Leave traces\nto allow cutting"
- note removed: "Vfb = 1.233V\nVo(min) = Vfb (R13 / R23 + 1)\nVo(max) = Vfb (R13 / R? + R13 / R23 + 1)"
- moved on the sheet: C1, C10, C11, C12, C13, C14, C15, C16, C17, C18, C19, C2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

Commit message: Fix PCB bug: FT2232 thermal pad too big
Other:
- note added: "V2 TODO: load vbus between 1uF and 10uF"
- moved on the sheet: C1, C10, C11, C12, C13, C14, C15, C16, C17, C18, C19, C2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
